File: GPT-E/Schede HW/Kicad/BatteryManagmentGPT-E/BatteryManagmentGPT-E.kicad_pcb (KiCad board)
At the start: 2 copper layers, 96.3 x 28.1 mm, 44 parts, among them J2 BATTERIA, J4 CONN_PCB, Q1 AO3401A, U3 LM393, U4 LMV7219M5

Commit message: update
Parts:
- removed SW: SWITCHxtelecomando, Connector_PinHeader_2.54mm:PinHeader_1x02_P2.54mm_Vertical
- removed USBC: Conn_01x04_Pin, Connector_Molex:Molex_KK-254_AE-6410-04A_1x04_P2.54mm_Vertical
- added J1: Conn_01x04_Pin, Connector_Molex:Molex_KK-254_AE-6410-04A_1x04_P2.54mm_Vertical, F.Cu at (112.9, 92.2)
- added J3: SWITCHxtelecomando, Connector_PinHeader_2.54mm:PinHeader_1x02_P2.54mm_Vertical, F.Cu at (195.2, 84.9)
- added R16: 2.2k, Resistor_THT:R_Axial_DIN0204_L3.6mm_D1.6mm_P5.08mm_Horizontal, F.Cu at (146.6, 100.9)
- moved R12 12.5 mm to (168.7, 89.5), turned to 0 degrees
Connections:
- C12 pad 1: Vref -> Net-(U1-K)
- R6 pad 2: Vref -> Net-(U1-K)
- U1 pad 1: Vref -> Net-(U1-K)
- U1 pad 2: Vref -> Net-(U1-K)
Routing:
- net V_ON: track 67.2 -> 52.5 mm, vias 0 -> 1
- net Vref: track 54.5 -> 47.2 mm
- net Net-(U1-K): track 0.00 -> 4.25 mm
- net Net-(D3-K): track 18.9 -> 20.4 mm
- added copper zone on F.Cu, net Net-(U1-K)
- removed copper zone on F.Cu, net Vref
