File: GPT-E/Schede HW/Kicad/BatteryManagmentGPT-E/BatteryManagmentGPT-E.kicad_sch (KiCad schematic)
At the start: 45 parts, among them J1 Conn_01x04_Pin, J2 BATTERIA, J3 SWITCHxtelecomando, J4 CONN_PCB, Q1 AO3401A, U3 LM393, U4 LMV7219M5

Commit message: update
Parts:
- J1: value Conn_01x04_Pin -> TPS4056
Other:
- moved on the sheet: H1, H3, H4
Changed lines of the file:
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@@
 	(symbol
 		(lib_id "Mechanical:MountingHole")
-		(at 16.51 99.06 0)
+		(at 16.51 125.73 0)
 		(unit 1)
 		(exclude_from_sim no)
@@
 		(on_board yes)
 		(dnp no)
-		(fields_autoplaced yes)
 		(property "Reference" "H1"
-			(at 19.05 97.7899 0)
+			(at 19.05 124.4599 0)
 			(effects
 				(font
@@
 		)
 		(property "Value" "MountingHole"
-			(at 19.05 100.3299 0)
+			(at 19.05 126.9999 0)
 			(effects
 				(font
@@
 		)
 		(property "Footprint" "MountingHole:MountingHole_2.2mm_M2"
-			(at 16.51 99.06 0)
+			(at 16.51 125.73 0)
 			(effects
 				(font
@@
 		)
 		(property "Datasheet" "~"
-			(at 16.51 99.06 0)
+			(at 16.51 125.73 0)
 			(effects
 				(font
@@
 		)
 		(property "Description" "Mounting Hole without connection"
-			(at 16.51 99.06 0)
+			(at 16.51 125.73 0)
 			(effects
 				(font
@@
 	(symbol
 		(lib_id "Mechanical:MountingHole")
-		(at 16.51 106.68 0)
+		(at 16.51 133.35 0)
 		(unit 1)
 		(exclude_from_sim no)
@@
 		(fields_autoplaced yes)
 		(property "Reference" "H3"
-			(at 19.05 105.4099 0)
+			(at 19.05 132.0799 0)
 			(effects
 				(font
@@
 		)
 		(property "Value" "MountingHole"
-			(at 19.05 107.9499 0)
+			(at 19.05 134.6199 0)
 			(effects
 				(font
@@
 		)
 		(property "Footprint" "MountingHole:MountingHole_2.2mm_M2"
-			(at 16.51 106.68 0)
+			(at 16.51 133.35 0)
 			(effects
 				(font
@@
 		)
 		(property "Datasheet" "~"
-			(at 16.51 106.68 0)
+			(at 16.51 133.35 0)
 			(effects
 				(font
@@
 		)
 		(property "Description" "Mounting Hole without connection"
-			(at 16.51 106.68 0)
+			(at 16.51 133.35 0)
 			(effects
 				(font
@@
 			)
 		)
-		(property "Value" "Conn_01x04_Pin"
+		(property "Value" "TPS4056"
 			(at 34.29 73.6599 0)
 			(effects
@@
 	(symbol
 		(lib_id "Mechanical:MountingHole")
-		(at 16.51 114.3 0)
+		(at 16.51 140.97 0)
 		(unit 1)
 		(exclude_from_sim no)
@@
 		(fields_autoplaced yes)
 		(property "Reference" "H4"
-			(at 19.05 113.0299 0)
+			(at 19.05 139.6999 0)
 			(effects
 				(font
@@
 		)
 		(property "Value" "MountingHole"
-			(at 19.05 115.5699 0)
+			(at 19.05 142.2399 0)
 			(effects
 				(font
@@
 		)
 		(property "Footprint" "MountingHole:MountingHole_2.2mm_M2"
-			(at 16.51 114.3 0)
+			(at 16.51 140.97 0)
 			(effects
 				(font
@@
 		)
 		(property "Datasheet" "~"
-			(at 16.51 114.3 0)
+			(at 16.51 140.97 0)
 			(effects
 				(font
@@
 		)
 		(property "Description" "Mounting Hole without connection"
-			(at 16.51 114.3 0)
-			(effects
-				(font
+			(at 16.51 140.97 0)
+			(effects
+				(font
