File: GPT-E/Schede HW/Kicad/HeadGPT-E/Head.kicad_sch (KiCad schematic)
At the start: 92 parts, among them J1 CH1, J10 CH3, J11 CH4, J12 CH5, J13 CH6, J14 CH9, J15 CH10, J16 CH11, J17 USBC, J18 SWITCH, J19 CH7, J2 STEREO, J20 CH8, J21 PANNELLO, J22 CH12, J3 I2C, J4 CH2, J5 BATTERIA, J6 SWITCH Batteria 11.1v, J7 CH0, J8 FAN, J9 PCA9685, Q2 IRLZ44N, Q3 2N7002, U1 FS8205A, U2 LM2596, U5 ESP32-DEVKITC-32D, U7 MAX98357A

Commit message: up
Parts:
- removed C15: 100uF, Capacitor_THT:CP_Radial_D5.0mm_P2.00mm, symbol Device:C_Polarized
- removed C9: 100nF, Capacitor_THT:C_Disc_D4.3mm_W1.9mm_P5.00mm, symbol Device:C
- removed D16: SS34, Diode_SMD:D_SMA_Handsoldering, symbol Diode:SS34
- removed J17: USBC, Connector_Molex:Molex_KK-254_AE-6410-04A_1x04_P2.54mm_Vertical, symbol Connector:Conn_01x04_Socket
- removed J6: SWITCH Batteria 11.1v, Connector_Molex:Molex_KK-254_AE-6410-02A_1x02_P2.54mm_Vertical, symbol Connector:Conn_01x02_Socket
- removed Q2: IRLZ44N, Package_TO_SOT_THT:TO-220-3_Vertical, symbol Transistor_FET:IRLZ44N
- removed Q3: 2N7002, Package_TO_SOT_SMD:SOT-23_Handsoldering, symbol Transistor_FET:2N7002
- removed R20: 470k, Resistor_THT:R_Axial_DIN0204_L3.6mm_D1.6mm_P5.08mm_Horizontal, symbol Device:R
- removed R23, R30: 10k, Resistor_THT:R_Axial_DIN0204_L3.6mm_D1.6mm_P5.08mm_Horizontal, symbol Device:R
- removed R24: 100k, Resistor_THT:R_Axial_DIN0204_L3.6mm_D1.6mm_P5.08mm_Horizontal, symbol Device:R
- removed R29: A1060, OptoDevice:R_LDR_D6.4mm_P3.4mm_Vertical, symbol Sensor_Optical:A1060
- removed U1: FS8205A, Package_SO:TSSOP-8_4.4x3mm_P0.65mm, symbol Libreria_Personale:FS8205A
- removed U5: ESP32-DEVKITC-32D, LIB_Personale:MODULE_ESP32-DEVKITC-32D, symbol Libreria_Personale:ESP32-DEVKITC-32D
- added C15, C21, C22: 100nF, Capacitor_THT:C_Disc_D4.3mm_W1.9mm_P5.00mm, symbol Device:C
- added C18, C9: 470uF, Capacitor_THT:CP_Radial_D5.0mm_P2.00mm, symbol Device:C_Polarized
- added C19: 100uF, Capacitor_THT:CP_Radial_D5.0mm_P2.00mm, symbol Device:C_Polarized
- added C20: 100n, Capacitor_THT:C_Disc_D4.3mm_W1.9mm_P5.00mm, symbol Device:C
- added D11: SMBJ12A, Diode_SMD:D_SMB_Handsoldering, symbol Diode:Z2SMBxxx
- added D17: SS34, Diode_SMD:D_SMA_Handsoldering, symbol Diode:SS34
- added J17: Conn_01x06_Socket, Connector_Molex:Molex_KK-254_AE-6410-06A_1x06_P2.54mm_Vertical, symbol Connector:Conn_01x06_Socket
- added J23: ~, Connector_Molex:Molex_Micro-Fit_3.0_43045-0400_2x02_P3.00mm_Horizontal, symbol Libreria_Personale:Conn._2x2_p3.0mm_horizontal
- added J6: UART, Connector_Molex:Molex_KK-254_AE-6410-03A_1x03_P2.54mm_Vertical, symbol Connector:Conn_01x03_Socket
- added Q1: BC547, Package_TO_SOT_THT:TO-92L_HandSolder, symbol Transistor_BJT:BC547
- added Q2: AO3401A, Package_TO_SOT_SMD:SOT-23W_Handsoldering, symbol Transistor_FET:AO3401A
- added R2: 10k, Resistor_THT:R_Axial_DIN0204_L3.6mm_D1.6mm_P5.08mm_Horizontal, symbol Device:R
- added U1: MINI360, LIB_Personale:Mini360, symbol Libreria_Personale:Mini360_DCDC_stepdown
- added U5: ESP32, LIB_Personale:ESP32, symbol Libreria_Personale:ESP32
- added U6: ~, symbol Libreria_Personale:TPS63020
- R11: value 100k -> 1k
- R17: value 10k -> 27k
Connections:
- net +3v3: now also C21.1, U1.3 (+Vout)
- net +5V: now also C15.1, C9.1, D17.1 (K), U1.1 (+Vin), U5.1 (VIN); no longer C4.1, U4.3 (VOUT+)
- net BAT+: now also J17.4 (Pin_4); no longer R11.1, U3.8 (BTP)
- net BAT+_ON: now also R11.1, U5.6 (D27); no longer R12.1
- net BAT+_RAW: now also U3.8 (BTP), J17.5 (Pin_5), Q2.2 (S), R2.2
- net BAT-: now also J17.3 (Pin_3)
- net BCLK: now also U5.9 (D33)
- net CHARGING: now also J17.6 (Pin_6)
- net DIN: now also U5.8 (D25)
- net GND: now also R17.1, C15.2, C18.2, C19.2, C20.2, C21.2, C22.2, C9.2, D11.2 (A), J17.1 (Pin_1), J17.2 (Pin_2), J23.1 (-), J23.3 (-), Q1.3 (E), U1.2 (-Vin), U1.4 (-Vout), U6.1 (GND), U6.2 (GND), U6.5 (GND), U6.6 (GND)
- net LRC: now also U5.10 (D32)
- net SCL: now also U5.17 (D22)
- net SDA: now also U5.20 (D21)
- net at J21.2 (Pin_2): now also C22.1, U6.3 (Vin), U6.4 (Vin)
- net power_11.1: now reaches D14.2 (A), J18.2 (Pin_2), R25.2
- net power_11.1: now also D10.2 (A)
- net 11.1v: now reaches C10.1, D9.1 (K), U2.1 (+IN)
- net 11.1v: now also R12.2
- net at R11.2: now also Q1.2 (B); no longer R17.2
- net at R31.2, R32.1: now also U5.14 (VP)
- net at D15.2 (A): now also U6.7 (Vout), U6.8 (Vout)
- net at D9.2 (A): now also C18.1, C19.1, C20.1, D11.1 (K), J23.2 (+), J23.4 (+)
- net +5v_11.1: no longer names the net of C3.1, J18.1 (Pin_1), R15.2, U2.3 (+OUT)
- net +5v_11.1: no longer D10.2 (A)
- net LDR_DX renamed LDR_panel
- net LDR_panel: now also U5.13 (VN)
- net LOAD: no longer names the net of C2.1, U4.1 (VIN+)
- net LOAD: now also Q2.3 (D)
- net Read_Battery for cutoff renamed Vsense3.7
- net Vsense3.7: now also U5.12 (D34)
- new net: Q1.1 (C), Q2.1 (G), R2.1
- new net: C4.1, D17.2 (A), U4.3 (VOUT+)
- new net RASPI_GND: J6.3 (Pin_3), U5.29 (GND2)
- new net UART_RX: J6.2 (Pin_2), U5.26 (D4)
- new net UART_TX: J6.1 (Pin_1), U5.23 (D5)
- new net Vsense11.1: R12.1, R17.2, U5.11 (D35)
- no-connect marks 13 -> 3
Other:
- note removed: "BRAIN_2"
- moved on the sheet: C1, C11, C12, C14, C16, C17, C2, C4, C5, C6, D10, D12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

Commit message: up
Other:
- moved on the sheet: J21
Changed lines of the file:
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@@
 	)
 	(junction
-		(at 187.96 58.42)
-		(diameter 0)
-		(color 0 0 0 0)
-	)
-	(junction
 		(at 44.45 43.18)
 		(diameter 0)
@@
 	)
 	(junction
+		(at 187.96 58.42)
+		(diameter 0)
+		(color 0 0 0 0)
+	)
+	(junction
 		(at 218.44 26.67)
 		(diameter 0)
@@
 	)
 	(junction
+		(at 185.42 58.42)
+		(diameter 0)
+		(color 0 0 0 0)
+	)
+	(junction
 		(at 54.61 50.8)
 		(diameter 0)
@@
 	(wire
 		(pts
-			(xy 181.61 34.29) (xy 181.61 67.31)
+			(xy 182.88 58.42) (xy 182.88 67.31)
 		)
 		(stroke
@@
 	(wire
 		(pts
+			(xy 185.42 58.42) (xy 187.96 58.42)
+		)
+		(stroke
+			(width 0)
+			(type default)
+		)
+	)
+	(wire
+		(pts
 			(xy 341.63 229.87) (xy 341.63 236.22)
 		)
@@
 	(wire
 		(pts
-			(xy 185.42 58.42) (xy 185.42 60.96)
-		)
-		(stroke
-			(width 0)
-			(type default)
-		)
-	)
-	(wire
-		(pts
 			(xy 53.34 62.23) (xy 53.34 64.77)
 		)
@@
 	(wire
 		(pts
-			(xy 181.61 67.31) (xy 187.96 67.31)
+			(xy 182.88 67.31) (xy 187.96 67.31)
 		)
 		(stroke
@@
 	(wire
 		(pts
-			(xy 187.96 58.42) (xy 185.42 58.42)
-		)
-		(stroke
-			(width 0)
-			(type default)
-		)
-	)
-	(wire
-		(pts
 			(xy 40.64 153.67) (xy 35.56 153.67)
 		)
@@
 	(wire
 		(pts
-			(xy 184.15 34.29) (xy 184.15 36.83)
+			(xy 185.42 58.42) (xy 185.42 59.69)
 		)
 		(stroke
@@
 	(symbol
 		(lib_id "Connector:Conn_01x02_Socket")
-		(at 184.15 29.21 270)
+		(at 185.42 53.34 270)
 		(mirror x)
 		(unit 1)
@@
 		(dnp no)
 		(property "Reference" "J21"
-			(at 184.1501 27.94 0)
+			(at 185.4201 52.07 0)
 			(effects
 				(font
@@
 		)
 		(property "Value" "PANNELLO"
-			(at 181.61 28.194 0)
+			(at 182.88 52.324 0)
 			(effects
 				(font
@@
 		)
 		(property "Footprint" "Connector_Molex:Molex_KK-254_AE-6410-02A_1x02_P2.54mm_Vertical"
-			(at 184.15 29.21 0)
+			(at 185.42 53.34 0)
 			(effects
 				(font
@@
 		)
 		(property "Datasheet" "~"
-			(at 184.15 29.21 0)
+			(at 185.42 53.34 0)
 			(effects
 				(font
@@
 		)
 		(property "Description" "Generic connector, single row, 01x02, script generated"
-			(at 184.15 29.21 0)
+			(at 185.42 53.34 0)
 			(effects
 				(font
@@
 	)
 	(symbol
-		(lib_id "power:GND")
-		(at 185.42 60.96 0)
-		(unit 1)
-		(exclude_from_sim no)
-		(in_bom yes)
-		(on_board yes)
-		(dnp no)
-		(property "Reference" "#PWR029"
-			(at 185.42 67.31 0)
-			(effects
-				(font
-					(size 1.27 1.27)
-				)
-				(hide yes)
-			)
-		)
-		(property "Value" "GND"
-			(at 185.42 65.278 0)
-			(effects
-				(font
-					(size 1.27 1.27)
-				)
-			)
-		)
-		(property "Footprint" ""
-			(at 185.42 60.96 0)
-			(effects
-				(font
-					(size 1.27 1.27)
-				)
-				(hide yes)
-			)
-		)
-		(property "Datasheet" ""
-			(at 185.42 60.96 0)
-			(effects
-				(font
-					(size 1.27 1.27)
-				)
-				(hide yes)
-			)
-		)
-		(property "Description" "Power symbol creates a global label with name \"GND\" , ground"
-			(at 185.42 60.96 0)
-			(effects
-				(font
-					(size 1.27 1.27)
-				)
-				(hide yes)
-			)
-		)
-		(pin "1"
-		)
-		(instances
-			(project "Head"
-				(path "/8e7ed3f4-22e2-435a-8dca-0a06eeede200"
-					(reference "#PWR029")
-					(unit 1)
-				)
-			)
-		)
-	)
-	(symbol
 		(lib_id "Diode:SS34")
 		(at 138.43 38.1 90)
@@
 	(symbol
 		(lib_id "power:GND")
-		(at 184.15 36.83 0)
+		(at 185.42 59.69 0)
 		(mirror y)
 		(unit 1)
@@
 		(dnp no)
 		(property "Reference" "#PWR05"
-			(at 184.15 43.18 0)
+			(at 185.42 66.04 0)
 			(effects
 				(font
@@
 		)
 		(property "Value" "GND"
-			(at 184.658 40.386 0)
+			(at 185.928 63.246 0)
 			(effects
 				(font
@@
 		)
 		(property "Footprint" ""
-			(at 184.15 36.83 0)
+			(at 185.42 59.69 0)
 			(effects
 				(font
@@
 		)
 		(property "Datasheet" ""
-			(at 184.15 36.83 0)
+			(at 185.42 59.69 0)
 			(effects
 				(font
@@
 		)
 		(property "Description" "Power symbol creates a global label with name \"GND\" , ground"
-			(at 184.15 36.83 0)
+			(at 185.42 59.69 0)
 			(effects
 				(font
