File: GPT-E/Schede HW/Kicad/HeadGPT-E/Head.kicad_sch (KiCad schematic)
At the start: 86 parts, among them J1 Right_Wheel_SERVO, J18 SWITCH, J2 STEREO, J3 I2C, J4 Left_Wheel SERVO, J5 Neck_SERVO2, J6 UARTtoRASPI, J7 Neck_SERVO1, J8 FAN, U1 LM3940-3.3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

Commit message: up
Parts:
- removed TP9: TestPoint, TestPoint:TestPoint_Pad_D1.5mm, symbol Connector:TestPoint
Changed lines of the file:
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@@
 	)
 	(junction
-		(at 179.07 165.1)
-		(diameter 0)
-		(color 0 0 0 0)
-	)
-	(junction
 		(at 217.17 101.6)
 		(diameter 0)
@@
 					(unit 1)
 				)
-			)
-		)
-	)
-	(symbol
-		(lib_id "Connector:TestPoint")
-		(at 179.07 165.1 0)
-		(unit 1)
-		(exclude_from_sim no)
-		(in_bom yes)
-		(on_board yes)
-		(dnp no)
-		(property "Reference" "TP9"
-			(at 177.546 159.766 0)
-			(effects
-				(font
-					(size 1.27 1.27)
-				)
-				(justify left)
-			)
-		)
-		(property "Value" "TestPoint"
-			(at 181.61 163.0679 0)
-			(effects
-				(font
-					(size 1.27 1.27)
-				)
-				(justify left)
-				(hide yes)
-			)
-		)
-		(property "Footprint" "TestPoint:TestPoint_Pad_D1.5mm"
-			(at 184.15 165.1 0)
-			(effects
-				(font
-					(size 1.27 1.27)
-				)
-				(hide yes)
-			)
-		)
-		(property "Datasheet" "~"
-			(at 184.15 165.1 0)
-			(effects
-				(font
-					(size 1.27 1.27)
-				)
-				(hide yes)
-			)
-		)
-		(property "Description" "test point"
-			(at 179.07 165.1 0)
-			(effects
-				(font
-					(size 1.27 1.27)
-				)
-				(hide yes)
-			)
-		)
-		(pin "1"
-		)
-		(instances
-			(project "Head"
-				(path "/8e7ed3f4-22e2-435a-8dca-0a06eeede200"
-					(reference "TP9")
-					(unit 1)
-				)

Commit message: update
Parts:
- removed C14: 470uF, Capacitor_THT:CP_Radial_D10.0mm_P5.00mm, symbol Device:C_Polarized
- added C10, C4: 100nF, Capacitor_SMD:C_0805_2012Metric_Pad1.18x1.45mm_HandSolder, symbol Device:C
- added C13: 1000uF, Capacitor_THT:CP_Radial_D12.5mm_P5.00mm, symbol Device:C_Polarized
- added R26: 10k, Resistor_SMD:R_1206_3216Metric_Pad1.30x1.75mm_HandSolder, symbol Device:R
- J2: value STEREO -> SPEAKER
Connections:
- net +3v3: now also C10.1, R26.1
- net +5V: now also C13.1, C4.1
- net Controllo_PCA: now also R26.2
- net GND: now also C10.2, C13.2, C4.2
Other:
- note added: "Se '1' uscite del pca disabilitate"
- note removed: "Se '0' uscite del pca disabilitate"
- moved on the sheet: C11, C12, C7, C8, R24
