File: GPT-E/Schede HW/Kicad/HeadGPT-E/Head.kicad_pcb (KiCad board)
At the start: 4 copper layers, 81.5 x 81.5 mm, 86 parts, among them J1 Right_Wheel_SERVO, J18 SWITCH, J2 STEREO, J3 I2C, J4 Left_Wheel SERVO, J5 Neck_SERVO2, J6 UARTtoRASPI, J7 Neck_SERVO1, J8 FAN, U1 LM3940-3.3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

Commit message: up
Parts:
- removed TP9: TestPoint, TestPoint:TestPoint_Pad_D1.5mm
Routing:
- net +5V: track 142.9 -> 105.0 mm
- net +3v3: track 8.85 -> 7.15 mm, vias 11 -> 10
- net 11.1v: track 43.7 -> 44.2 mm
Changed lines of the file:
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@@
 		)
 	)
-	(footprint "TestPoint:TestPoint_Pad_D1.5mm"
-		(layer "F.Cu")
-		(at 142.4 68.28)
-		(descr "SMD pad as test Point, diameter 1.5mm")
-		(tags "test point SMD pad")
-		(property "Reference" "TP9"
-			(at 0 -1.648 0)
-			(layer "F.SilkS")
-			(effects
-				(font
-					(size 1 1)
-					(thickness 0.15)
-				)
-			)
-		)
-		(property "Value" "TestPoint"
-			(at 0 1.75 0)
-			(layer "F.Fab")
-			(effects
-				(font
-					(size 1 1)
-					(thickness 0.15)
-				)
-			)
-		)
-		(property "Datasheet" "~"
-			(at 0 0 0)
-			(unlocked yes)
-			(layer "F.Fab")
-			(hide yes)
-			(effects
-				(font
-					(size 1.27 1.27)
-					(thickness 0.15)
-				)
-			)
-		)
-		(property "Description" "test point"
-			(at 0 0 0)
-			(unlocked yes)
-			(layer "F.Fab")
-			(hide yes)
-			(effects
-				(font
-					(size 1.27 1.27)
-					(thickness 0.15)
-				)
-			)
-		)
-		(property ki_fp_filters "Pin* Test*")
-		(sheetname "/")
-		(sheetfile "Head.kicad_sch")
-		(attr exclude_from_pos_files)
-		(fp_circle
-			(center 0 0)
-			(end 0 0.95)
-			(stroke
-				(width 0.12)
-				(type solid)
-			)
-			(fill no)
-			(layer "F.SilkS")
-		)
-		(fp_circle
-			(center 0 0)
-			(end 1.25 0)
-			(stroke
-				(width 0.05)
-				(type solid)
-			)
-			(fill no)
-			(layer "F.CrtYd")
-		)
-		(fp_text user "${REFERENCE}"
-			(at 0 -1.65 0)
-			(layer "F.Fab")
-			(effects
-				(font
-					(size 1 1)
-					(thickness 0.15)
-				)
-			)
-		)
-		(pad "1" smd circle
-			(at 0 0)
-			(size 1.5 1.5)
-			(layers "F.Cu" "F.Mask")
-			(net 5 "+3v3")
-			(pinfunction "1")
-			(pintype "passive")
-		)
-		(embedded_fonts no)
-	)
 	(footprint "Capacitor_SMD:C_0805_2012Metric_Pad1.18x1.45mm_HandSolder"
 		(layer "F.Cu")
@@
 	)
 	(segment
-		(start 132.51 63.18)
-		(end 137.21 58.48)
-		(width 1.5)
-		(layer "F.Cu")
-		(net 4)
-	)
-	(segment
 		(start 145.54 122.65)
 		(end 138.889875 122.65)
@@
 	)
 	(segment
-		(start 128.857677 53.71)
-		(end 132.44 53.71)
-		(width 1.5)
-		(layer "F.Cu")
-		(net 4)
-	)
-	(segment
 		(start 120.79 118.58)
 		(end 118.38 118.58)
@@
 	)
 	(segment
-		(start 132.44 53.71)
-		(end 137.21 58.48)
-		(width 1.5)
-		(layer "F.Cu")
-		(net 4)
-	)
-	(segment
 		(start 99.8575 100.36)
 		(end 99.365 100.36)
@@
 	)
 	(segment
-		(start 119.087677 53.46)
-		(end 117.397677 53.46)
-		(width 1.5)
-		(layer "F.Cu")
-		(net 4)
-	)
-	(segment
-		(start 119.197677 63.21)
-		(end 117.287677 63.21)
-		(width 1.5)
-		(layer "F.Cu")
-		(net 4)
-	)
-	(segment
-		(start 128.927677 63.18)
-		(end 132.51 63.18)
-		(width 1.5)
-		(layer "F.Cu")
-		(net 4)
-	)
-	(segment
 		(start 120.5 122.8)
 		(end 119.89 123.41)
@@
 	)
 	(segment
-		(start 117.397677 53.46)
-		(end 112.467677 58.39)
-		(width 1.5)
-		(layer "F.Cu")
-		(net 4)
-	)
-	(segment
-		(start 117.287677 63.21)
-		(end 112.467677 58.39)
-		(width 1.5)
-		(layer "F.Cu")
-		(net 4)
-	)
-	(segment
 		(start 93.74 97.1425)
 		(end 96.1475 97.1425)
@@
 	)
 	(segment
-		(start 142.4 68.28)
-		(end 142.4 69.98)
-		(width 0.5)
-		(layer "F.Cu")
-		(net 5)
-	)
-	(segment
 		(start 131.67 94.37)
 		(end 131.67 93.28)
@@
 	)
 	(via
-		(at 142.4 69.98)
-		(size 0.6)
-		(drill 0.3)
-		(layers "F.Cu" "B.Cu")
-		(net 5)
-	)
-	(via
 		(at 107.41 104.1)
 		(size 0.6)
@@
 	(segment
 		(start 87.07 73.96)
-		(end 89.0675 73.96)
+		(end 89.975 73.96)
 		(width 1.5)
 		(layer "F.Cu")
@@
 	)
 	(segment
-		(start 89.0675 73.96)
-		(end 90.1075 75)
-		(width 1.5)
+		(start 90.0025 77.2425)
+		(end 90.075 77.17)
+		(width 1)
 		(layer "F.Cu")
 		(net 6)
 	)
 	(segment
-		(start 90.0025 77.2425)
-		(end 90.075 77.17)
-		(width 1)
+		(start 90.1075 74.0925)
+		(end 90.1075 75)
+		(width 1.5)
 		(layer "F.Cu")
 		(net 6)
@@
 		(width 1.5)
 		(layer "F.Cu")
+		(net 6)
+	)
+	(segment
+		(start 89.975 73.96)
+		(end 90.1075 74.0925)
+		(width 1.5)
+		(layer "F.Cu")

Commit message: update
Parts:
- removed C14: 470uF, Capacitor_THT:CP_Radial_D10.0mm_P5.00mm
- added C10: 100nF, Capacitor_SMD:C_0805_2012Metric_Pad1.18x1.45mm_HandSolder, F.Cu at (107.3, 99.4)
- added C13: 1000uF, Capacitor_THT:CP_Radial_D12.5mm_P5.00mm, F.Cu at (108.9, 56.9)
- added C4: 100nF, Capacitor_SMD:C_0805_2012Metric_Pad1.18x1.45mm_HandSolder, F.Cu at (96.2, 99.9)
- added R26: 10k, Resistor_SMD:R_1206_3216Metric_Pad1.30x1.75mm_HandSolder, F.Cu at (131.9, 89.2)
- J2: value STEREO -> SPEAKER
- moved TP1 28.8 mm to (101.7, 76.3)
- moved R15 11.4 mm to (83.7, 84.7), turned to 0 degrees
- moved R20 10.7 mm to (83.0, 76.6)
- moved R11 6.76 mm to (86.3, 89.4)
- moved C21 4.75 mm to (82.2, 79.4), turned to -90 degrees
- moved C8 2.20 mm to (109.4, 99.4)
- moved D6 1.84 mm to (146.6, 124.9)
- moved D5 1.23 mm to (137.0, 124.9)
- moved C7 1.11 mm to (96.2, 96.0)
- moved D8 0.65 mm to (127.4, 125.0)
Routing:
- net GND: track 71.9 -> 83.8 mm, vias 23 -> 24
- net Net-(U2-FB): track 14.8 -> 5.89 mm
- net +5V: track 105.0 -> 112.1 mm, vias 13 -> 14
- net Net-(U2-COMP): track 4.54 -> 10.1 mm, vias 0 -> 2
- net Net-(D5-RK): track 9.65 -> 8.33 mm
- net +3v3: track 7.15 -> 8.40 mm, vias 10 -> 11
- net Net-(D6-GK): track 11.0 -> 10.2 mm
- net Net-(D8-GK): track 13.9 -> 13.4 mm
- net Net-(D5-BK): track 9.82 -> 9.30 mm
