File: TranslateIA/TranslateIA.kicad_sch (KiCad schematic)
At the start: 36 parts, among them J2 BATTERIA, J2 TPS4056, Q1 AO3401A, SW1 SW_Push_Dual, SW2 SW_Push_Dual, U1 MAX98357A, U2 ESP32, U3 MT3608, U4 Raspberry Pi Zero 2 W, U5 AMS1117-3.3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

Commit message: updated
Parts:
- removed C10: 220uF, Capacitor_THT:CP_Radial_D5.0mm_P2.00mm, symbol Device:C_Polarized
- removed C4, C5: 100nF, Capacitor_THT:C_Disc_D4.3mm_W1.9mm_P5.00mm, symbol Device:C
- removed U1: MAX98357A, Package_DFN_QFN:TDFN-14-1EP_3x3mm_P0.4mm_EP1.78x2.35mm_ThermalVias, symbol Libreria_Personale:MAX98357A
- removed U3: MT3608, LIB_Personale:MT3608-Module, symbol Libreria_Personale:MT3608
- removed U5: AMS1117-3.3, Package_TO_SOT_SMD:SOT-223-3_TabPin2, symbol Regulator_Linear:AMS1117-3.3
- added J1: Display OLED, Connector_Molex:Molex_KK-254_AE-6410-04A_1x04_P2.54mm_Vertical, symbol Connector:Conn_01x04_Pin
- added R10, R8, R9: 330, Resistor_THT:R_Axial_DIN0204_L3.6mm_D1.6mm_P5.08mm_Horizontal, symbol Device:R
- added R11, R12: 10k, Resistor_THT:R_Axial_DIN0204_L3.6mm_D1.6mm_P5.08mm_Horizontal, symbol Device:R
- added U1: PCM5102A, LIB_Personale:PCM5102A, symbol Libreria_Personale:PCM5102A
- added U5: XL6009, LIB_Personale:LM2896, symbol Libreria_Personale:XL6009
- C9: value 220uF -> 1000uF
- SW1, SW2: footprint (none) -> Button_Switch_THT:Push_E-Switch_KS01Q01
- renumbered J2 to J3
Connections:
- net +3v3_ESP: now also R11.1, R12.1
- net +5v: now also C12.1, U6.1 (+Vin), J1.2 (Pin_2), U1.1 (Vcc), U5.3 (+OUT)
- net BCLK: now also U1.7 (BCK)
- net DIN: now also U1.8 (DIN)
- net GND: now also C6.2, D2.1 (K), D3.1 (K), D4.1 (K), SW1.1, SW2.1, J1.1 (Pin_1), U1.10 (FMT), U1.3 (GND), U1.6 (SCL), U5.2 (-IN), U5.4 (-OUT); no longer C6.1
- net LRC: now also U1.9 (LCK)
- net pwmB: now also U2.3 (D13)
- net pwmG: now also U2.5 (D14)
- net pwmR: now also U2.6 (D27)
- net TXesp: now reaches U4.10 (GPIO15-UARTrx)
- net TXesp: now also U2.18 (TX0)
- net RXesp: now reaches U4.8 (GPIO14-UARTtx)
- net RXesp: now also U2.19 (RX0)
- net at D2.2 (A): now also R8.2
- net at U2.16 (D23): now also R10.1
- net SCL: now reaches U2.17 (D22)
- net SCL: now also J1.3 (Pin_3), R12.2
- net SDA: now reaches U2.20 (D21)
- net SDA: now also J1.4 (Pin_4), R11.2
- net Button>: now reaches U2.21 (D19)
- net Button>: now also SW1.4
- net Button<: now reaches U2.22 (D18)
- net Button<: now also SW2.4
- net at U2.23 (D5): now also R9.1
- net at U2.26 (D4): now also R8.1
- net at D4.2 (A): now also R10.2
- net at D3.2 (A): now also R9.2
- new net: C6.1, D5.1 (K), Q1.3 (D), U5.1 (+IN)
- no-connect marks 2 -> 50
Other:
- moved on the sheet: C11, C12, C6, C7, C9, D1, D2, D3, D4, R5, R6, R7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

Commit message: up
Parts:
- added M1: INMP441, LIB_Personale:INMP441, symbol Libreria_Personale:INMP441_Microphone_I2S
Connections:
- net +3v3_ESP: no longer C11.1, C8.1, U2.1 (VIN), U6.3 (+Vout)
- net GND: now also M1.GND, M1.L/R
- net RXesp: now also U2.25 (RX2); no longer U2.19 (RX0)
- net TXesp: now also U2.24 (TX2); no longer U2.18 (TX0)
- net SD: now reaches U2.13 (VN)
- net SD: now also M1.SD
- net SCK: now reaches U2.28 (D15)
- net SCK: now also M1.SCK
- net WS: now reaches U2.7 (D26)
- net WS: now also M1.WS
- new net +3v3: C11.1, C8.1, M1.VDD, U2.1 (VIN), U6.3 (+Vout)
- no-connect marks 50 -> 47
