File: TranslateIA/Schematico/TranslateIA.kicad_sch (KiCad schematic)
At the start: 39 parts, among them J1 Display OLED, J2 TPS4056, J3 BATTERIA, M1 INMP441, Q1 AO3401A, SW1 SW_Push_Dual, SW2 SW_Push_Dual, U1 PCM5102A, U2 ESP32, U4 Raspberry Pi Zero 2 W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

Commit message: up
Parts:
- added J4: switch, Connector_Molex:Molex_KK-254_AE-6410-02A_1x02_P2.54mm_Vertical, symbol Connector:Conn_01x02_Socket
- added R13, R14: 220, Resistor_THT:R_Axial_DIN0204_L3.6mm_D1.6mm_P5.08mm_Horizontal, symbol Device:R
- added R15, R16, R17: 33, Resistor_THT:R_Axial_DIN0204_L3.6mm_D1.6mm_P5.08mm_Horizontal, symbol Device:R
- added SW3: SW_Push_Dual, Button_Switch_THT:Push_E-Switch_KS01Q01, symbol Switch:SW_Push_Dual
- R11, R12: value 10k -> 4.7k
Connections:
- net BCLK: now also R15.1; no longer U2.9 (D33)
- net GND: now also SW3.1
- net LRC: now also R17.1; no longer U2.10 (D32)
- net RXesp: now also R14.2; no longer U2.25 (RX2)
- net SCK: now also R16.2; no longer U2.28 (D15)
- net TXesp: now also R13.2; no longer U2.24 (TX2)
- net at C6.1, U5.1 (+IN): now also J4.1 (Pin_1); no longer D5.1 (K), Q1.3 (D)
- net ok: now reaches U2.14 (VP)
- net ok: now also SW3.4
- new net: R14.1, U2.25 (RX2)
- new net: R17.2, U2.10 (D32)
- new net: R13.1, U2.24 (TX2)
- new net: R16.1, U2.28 (D15)
- new net: R15.2, U2.9 (D33)
- new net: D5.1 (K), J4.2 (Pin_2), Q1.3 (D)
- no-connect marks 47 -> 48
Other:
- moved on the sheet: J1, R11, R12, SW1, SW2, U1
