File: TranslateIA/Schematico/TranslateIA.kicad_sch (KiCad schematic)
At the start: 63 parts, among them IC1 MP2307DN-LF, J2 speaker, J3 battery, J4 switch, J5 dnp, J6 uart, J7 uart, M1 INMP441, Q1 AO3401A, SW1 SW_Push_Dual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

Commit message: update
Parts:
- removed C2: 220uF, Capacitor_THT:CP_Radial_D5.0mm_P2.00mm, symbol Device:C_Polarized
- removed D5: 1N5819, Diode_THT:D_DO-41_SOD81_P7.62mm_Horizontal, symbol Diode:1N5819
- added C15, C18, C2: 100nF, Capacitor_SMD:C_0805_2012Metric_Pad1.18x1.45mm_HandSolder, symbol Device:C
- added C16, C17, C19, C20: 10uF, Capacitor_SMD:C_0805_2012Metric_Pad1.18x1.45mm_HandSolder, symbol Device:C
- added F1: Fuse_Small, Fuse:Fuseholder_Littelfuse_Nano2_154x, symbol Device:Fuse_Small
- C1, C11, C12, C14, C3, C5: footprint Capacitor_THT:C_Disc_D4.3mm_W1.9mm_P5.00mm -> Capacitor_SMD:C_0805_2012Metric_Pad1.18x1.45mm_HandSolder
- C4: footprint Capacitor_THT:CP_Radial_D5.0mm_P2.00mm -> Capacitor_SMD:C_0805_2012Metric_Pad1.18x1.45mm_HandSolder
- R4: value 100k -> 220k
Connections:
- net +3v3: now also C17.1, C18.1, C20.1
- net +5v: now also C15.1, C16.1, C19.1
- net BAT+: now also F1.2; no longer Q1.2 (S)
- net GND: now also C15.2, C16.2, C17.2, C18.2, C19.2, C2.2, C20.2
- net Vsense: now also C2.1
- net at C4.1, IC1.2 (IN), J4.1 (Pin_1)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: now also C5.1
- net at J4.2 (Pin_2): now also Q1.2 (S); no longer Q1.3 (D)
- net Vbus: no longer names the net of Q1.1 (G), R2.1
- net Vbus: no longer C5.1, U5.1 (+)
- new net 7v4: F1.1, Q1.3 (D)
- new net USB_Vbus: U5.1 (+)
Other:
- moved on the sheet: C8, C9, R3, R4, U5
