File: TranslateIA/Schematico/TranslateIA.kicad_pcb (KiCad board)
At the start: 4 copper layers, 85.5 x 112.2 mm, 71 parts, among them IC1 MP2307DN-LF, J2 speaker, J3 battery, J4 switch, J5 dnp, J6 uart, J7 uart, M1 INMP441, Q1 AO3401A, SW1 SW_Push_Dual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

Commit message: update
Parts:
- removed D5: 1N5819, Diode_THT:D_DO-41_SOD81_P7.62mm_Horizontal
- added C15: 100nF, Capacitor_SMD:C_0805_2012Metric_Pad1.18x1.45mm_HandSolder, F.Cu at (84.3, 80.0)
- added C16: 10uF, Capacitor_SMD:C_0805_2012Metric_Pad1.18x1.45mm_HandSolder, F.Cu at (82.1, 80.0)
- added C17: 10uF, Capacitor_SMD:C_0805_2012Metric_Pad1.18x1.45mm_HandSolder, F.Cu at (140.8, 47.9)
- added C18: 100nF, Capacitor_SMD:C_0805_2012Metric_Pad1.18x1.45mm_HandSolder, F.Cu at (142.9, 47.9)
- added C19: 10uF, Capacitor_SMD:C_0805_2012Metric_Pad1.18x1.45mm_HandSolder, F.Cu at (106.7, 62.8)
- added C20: 10uF, Capacitor_SMD:C_0805_2012Metric_Pad1.18x1.45mm_HandSolder, F.Cu at (106.5, 87.0)
- added F1: Fuse_Small, Fuse:Fuseholder_Littelfuse_Nano2_154x, F.Cu at (100.5, 30.7)
- C1, C11, C12, C14, C3, C5: footprint Capacitor_THT:C_Disc_D4.3mm_W1.9mm_P5.00mm -> Capacitor_SMD:C_0805_2012Metric_Pad1.18x1.45mm_HandSolder
- C2: value 220uF -> 100nF; footprint Capacitor_THT:CP_Radial_D5.0mm_P2.00mm -> Capacitor_SMD:C_0805_2012Metric_Pad1.18x1.45mm_HandSolder
- C4: footprint Capacitor_THT:CP_Radial_D5.0mm_P2.00mm -> Capacitor_SMD:C_0805_2012Metric_Pad1.18x1.45mm_HandSolder
- R4: value 100k -> 220k
- moved C2 52.6 mm to (122.9, 70.4), turned to 90 degrees
- moved C5 50.6 mm to (96.1, 40.3), turned to 90 degrees
- moved C4 11.7 mm to (92.9, 28.5), turned to 0 degrees
- moved R2 10.3 mm to (112.9, 24.6), turned to 0 degrees
- moved C12 7.00 mm to (106.7, 65.0), turned to 0 degrees
- moved Q1 4.81 mm to (108.3, 25.5)
- moved C11 3.97 mm to (106.5, 84.9)
- moved C9 3.44 mm to (81.4, 84.3), turned to -90 degrees
- moved C14 2.46 mm to (96.1, 44.2)
- moved C1 1.09 mm to (135.8, 61.2)
- moved C8 0.91 mm to (145.5, 40.8)
- moved C3 0.85 mm to (130.7, 61.1)
Connections:
- C2 pad 1: Vbus -> Vsense
- C5 pad 1: Vbus -> Net-(IC1-IN)
- J4 pad 2: Net-(D5-K) -> Net-(J4-Pin_2)
- Q1 pad 1: Vbus -> Net-(Q1-G)
- Q1 pad 2: BAT+ -> Net-(J4-Pin_2)
- Q1 pad 3: Net-(D5-K) -> /7v4
- R2 pad 1: Vbus -> Net-(Q1-G)
- U5 pad 1: Vbus -> USB_Vbus
Routing:
- net GND: track 14.1 -> 52.0 mm, vias 7 -> 11
- net Net-(D5-K): track 35.4 -> 0.00 mm
- net Net-(J4-Pin_2): track 0.00 -> 22.9 mm
- net BAT+: track 82.3 -> 67.1 mm, vias 0 -> 4
- net /7v4: track 0.00 -> 12.7 mm
- net +3v3: track 5.62 -> 17.1 mm
- net DIN: track 42.7 -> 51.8 mm
- net +5v: track 1.55 -> 8.88 mm
- net Net-(IC1-SW): track 16.8 -> 12.1 mm
- net Net-(IC1-IN): track 55.2 -> 52.0 mm
- net SD: track 52.5 -> 55.3 mm
- net Net-(Q1-G): track 0.00 -> 2.15 mm
- net Net-(IC1-BS): track 6.07 -> 5.42 mm, vias 0 -> 2
- removed copper zone on F.Cu, net Vbus
