File: GPT-E/Schede HW/Kicad/TelecomandoGPT-E/File KiCad/Telecomando_ROBOT.kicad_pcb (KiCad board)
At the start: 4 copper layers, 149.3 x 51.5 mm, 46 parts, among them J1 Conn_01x02, J2 Conn_01x02, J4 USB_C_Receptacle_USB2.0_16P, M1 INMP441, M2 INMP441, SW1 SW_Push_Open_Dual, SW2 SX, SW3 DX, SW4 OK, SW5 PUSH_TO_TALK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

Commit message: UP
Parts:
- J1, J2: footprint Connector_Molex:Molex_KK-254_AE-6410-02A_1x02_P2.54mm_Vertical -> Connector_JST:JST_EH_B2B-EH-A_1x02_P2.50mm_Vertical
- moved TP1 5.61 mm to (149.2, 113.6)
- moved TP6 5.52 mm to (146.5, 113.6)
- moved J2 2.28 mm to (149.8, 109.6)
- moved TP2 1.32 mm to (151.8, 113.5)
Connections:
- D1 pad 1: GND -> Net-(D1-K)
- D1 pad 2: Net-(D1-RA) -> GND
- R1 pad 2: Net-(D1-RA) -> Net-(D1-K)
Routing:
- net D+: track 16.2 -> 22.2 mm
- net Net-(D1-RA): track 5.62 -> 0.00 mm
- net Net-(D1-K): track 0.00 -> 4.77 mm
- net Batteria: track 71.2 -> 67.4 mm
- net D-: track 16.8 -> 17.8 mm
- net GND: vias 280 -> 284
