File: GPT-E/Schede HW/Kicad/TelecomandoGPT-E/File KiCad/Telecomando_ROBOT.kicad_sch (KiCad schematic)
At the start: 46 parts, among them J1 Conn_01x02, J2 Conn_01x02, J4 USB_C_Receptacle_USB2.0_16P, M1 INMP441, M2 INMP441, SW1 SW_Push_Open_Dual, SW2 SX, SW3 DX, SW4 OK, SW5 PUSH_TO_TALK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

Commit message: UP
Connections:
- net GND: now also D1.2 (K); no longer D1.1 (K)
- net at R1.2: now also D1.1 (RA); no longer D1.2 (RA)
