File: GPT-E/Schede HW/Kicad/PowerManagement_GPT-E/PowerManagement_GPT-E.kicad_pcb (KiCad board)
At the start: 2 copper layers, 161.5 x 66.9 mm, 71 parts, among them J1 Battery, J2 switch, J3 Conn_01x02_Socket, J4 Conn_02x02_Counter_Clockwise, J5 Conn_01x02, J6 Conn_01x02, J7 Charge_conn, J8 Voltage_indicator, J9 Buzzer_Accensione, Q1 IRLZ44N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

Commit message: up
Parts:
- moved R3 14.2 mm to (209.9, 82.0)
Connections:
- U1 pad 4: unconnected-(U1-PD2-Pad4) -> Net-(U1-PD2)
- U3 pad 8: unconnected-(U3-IRQ-Pad8) -> Net-(U1-PD2)
Routing:
- net Net-(U1-PD2): track 0.00 -> 48.9 mm, vias 0 -> 1
- net Net-(U1-PC6/~{RESET}): track 14.0 -> 2.56 mm
