File: GPT-E/Schede HW/Kicad/PowerManagement_GPT-E/PowerManagement_GPT-E.kicad_pcb (KiCad board)
At the start: 2 copper layers, 161.5 x 66.9 mm, 71 parts, among them J1 Battery, J2 switch, J3 Conn_01x02_Socket, J4 Conn_02x02_Counter_Clockwise, J5 Conn_01x02, J6 Conn_01x02, J7 Charge_conn, J8 Voltage_indicator, J9 Buzzer_Accensione, Q1 IRLZ44N, Q2 IRF7416TRPBF, SW1 SW_SPDT, U1 ATmega8-16P, U2 BMS_3S_LithiumBattery18650, U3 NRF24L01_Breakout, U4 LM393, U5 MP1584, Y1 16MHz

Commit message: up
Parts:
- removed C15: 22u, Capacitor_THT:CP_Radial_D6.3mm_P2.50mm
- removed C38, C40: C_Polarized, Capacitor_THT:CP_Radial_D6.3mm_P2.50mm
- removed C39: C, Capacitor_THT:C_Disc_D5.1mm_W3.2mm_P5.00mm
- removed Cbypass1, Crc1, Crc2: 100n, Capacitor_THT:C_Disc_D5.1mm_W3.2mm_P5.00mm
- removed J5, J6: Conn_01x02, Connector_Molex:Molex_KK-254_AE-6410-02A_1x02_P2.54mm_Vertical
- removed J8: Voltage_indicator, Connector_PinHeader_2.54mm:PinHeader_1x09_P2.54mm_Vertical
- removed J9: Buzzer_Accensione, Connector:FanPinHeader_1x03_P2.54mm_Vertical
- removed Ra1, Ra3, Rb5, Rb6: 22k, Resistor_THT:R_Axial_DIN0204_L3.6mm_D1.6mm_P5.08mm_Horizontal
- removed Ra2, Ra4, Rb2, Rb4: 10k, Resistor_THT:R_Axial_DIN0204_L3.6mm_D1.6mm_P5.08mm_Horizontal
- removed Rb1, Rb3: 47k, Resistor_THT:R_Axial_DIN0204_L3.6mm_D1.6mm_P5.08mm_Horizontal
- removed Rf1, Rf2: Rfb, Resistor_THT:R_Axial_DIN0204_L3.6mm_D1.6mm_P5.08mm_Horizontal
- removed TPVref1, TPsupply1: TestPoint, TestPoint:TestPoint_Pad_2.0x2.0mm
- removed U4: LM393, Package_DIP:DIP-8_W7.62mm
- removed U8: ~, LIB_Personale:Mini360
- added BZ1: TMB12A03, Buzzer_Beeper:Buzzer_12x9.5RM7.6, F.Cu at (158.3, 96.7)
- added C11: 100n, Capacitor_SMD:C_0805_2012Metric_Pad1.18x1.45mm_HandSolder, F.Cu at (153.0, 106.7)
- added D5: BZT52C12, Diode_SMD:D_SOD-123, F.Cu at (151.7, 77.8)
- added Q3: AO4407, Package_SO:SOIC-8_3.9x4.9mm_P1.27mm, F.Cu at (159.9, 75.0)
- added Q4: BC547, Package_TO_SOT_THT:TO-92L_Inline, F.Cu at (167.5, 89.2)
- added R10: 100K, Resistor_THT:R_Axial_DIN0204_L3.6mm_D1.6mm_P5.08mm_Horizontal, F.Cu at (145.9, 115.4)
- added R8: 100K, Resistor_SMD:R_1206_3216Metric_Pad1.30x1.75mm_HandSolder, F.Cu at (143.4, 73.7)
- added R9: 4.7k, Resistor_SMD:R_1206_3216Metric_Pad1.30x1.75mm_HandSolder, F.Cu at (172.8, 88.1)
- added TPbat+1: TestPoint, TestPoint:TestPoint_Pad_2.0x2.0mm, F.Cu at (123.8, 79.1)
- added TPload1: TestPoint, TestPoint:TestPoint_Pad_2.0x2.0mm, F.Cu at (163.1, 57.0)
- C1, C10, C3, C5, C8, C9: footprint Capacitor_THT:C_Disc_D7.0mm_W2.5mm_P5.00mm -> Capacitor_SMD:C_0805_2012Metric_Pad1.18x1.45mm_HandSolder
- C2: value 10u -> 10uF; footprint Capacitor_THT:CP_Radial_D8.0mm_P3.50mm -> Capacitor_SMD:C_0805_2012Metric_Pad1.18x1.45mm_HandSolder
- C6: value 100n -> 10uF; footprint Capacitor_THT:C_Disc_D7.0mm_W2.5mm_P5.00mm -> Capacitor_SMD:C_0805_2012Metric_Pad1.18x1.45mm_HandSolder
- C7: value 100u -> 10uF; footprint Capacitor_THT:CP_Radial_D8.0mm_P3.50mm -> Capacitor_SMD:C_0805_2012Metric_Pad1.18x1.45mm_HandSolder
- J3: value Conn_01x02_Socket -> Conn_02x02_Counter_Clockwise; footprint Connector_PinSocket_2.54mm:PinSocket_1x02_P2.54mm_Vertical -> Connector_Molex:Molex_Micro-Fit_3.0_43045-0412_2x02_P3.00mm_Vertical
- Q1: value IRLZ44N -> BC547; footprint Package_TO_SOT_THT:TO-220-3_Horizontal_TabDown -> Package_TO_SOT_THT:TO-92L_Inline
- R1: value 100 -> 4.7k; footprint Resistor_THT:R_Axial_DIN0204_L3.6mm_D1.6mm_P5.08mm_Horizontal -> Resistor_SMD:R_1206_3216Metric_Pad1.30x1.75mm_HandSolder
- R11: value 10k -> 33k
- R2: value 100k -> 100K; footprint Resistor_THT:R_Axial_DIN0204_L3.6mm_D1.6mm_P5.08mm_Horizontal -> Resistor_SMD:R_1206_3216Metric_Pad1.30x1.75mm_HandSolder
- R4: value 1k -> 2.2k
- R6: value 10k -> 100; footprint Resistor_THT:R_Axial_DIN0204_L3.6mm_D1.6mm_P5.08mm_Horizontal -> Resistor_SMD:R_1206_3216Metric_Pad1.30x1.75mm_HandSolder
- U5: value MP1584 -> AZ1117CH2-3.3; footprint Converter_DCDC:MP1584 -> Package_TO_SOT_SMD:SOT-223-3_TabPin2
- Y1: value 16MHz -> 8MHz
- moved R11 50.9 mm to (140.9, 117.7)
- moved C3 49.5 mm to (190.3, 101.8), turned to 0 degrees
- moved EN1 40.1 mm to (138.1, 91.8)
- moved Q1 35.6 mm to (146.2, 77.3)
- moved R1 35.0 mm to (145.0, 93.0)
- moved R2 31.3 mm to (154.4, 77.8), turned to -90 degrees
- moved SW1 28.5 mm to (148.6, 92.0), turned to 0 degrees
- moved D2 27.6 mm to (211.3, 77.3), turned to 0 degrees
- moved R4 24.3 mm to (208.2, 77.3), turned to 90 degrees
- moved C8 24.1 mm to (136.5, 112.4), turned to -90 degrees
- moved J4 19.7 mm to (183.7, 64.5)
- moved Q2 18.3 mm to (137.2, 101.4)
- moved R6 16.0 mm to (149.2, 77.8), turned to -90 degrees
- moved C7 15.8 mm to (150.8, 106.7)
- moved C9 14.2 mm to (181.4, 82.8), turned to 0 degrees
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Connections:
- C1 pad 1: Net-(U1-AVCC) -> +3v3
- C1 pad 2: +3v3 -> GND
- C12 pad 1: IN -> +v
- C3 pad 1: Net-(Q1-G) -> Net-(U1-AREF)
- C4 pad 1: +v -> LOAD
- C4 pad 2: Net-(D1-A) -> GND
- C6 pad 1: GND -> +bat
- C6 pad 2: BATT+ -> GND
- C8 pad 1: +3v3 -> +bat
- D1 pad 1: +v -> LOAD
- D1 pad 2: Net-(D1-A) -> GND
- D2 pad 2: Net-(D1-A) -> GND
- J2 pad 1: BATT+ -> +bat
- J2 pad 2: IN -> +v
- J3 pad 1: Net-(D1-A) -> GND
- J3 pad 2: +v -> LOAD
- J4 pad 1: Net-(D1-A) -> GND
- J4 pad 2: +v -> LOAD
- J4 pad 3: Net-(D1-A) -> GND
- J4 pad 4: +v -> LOAD
- Q1 pad 1: Net-(Q1-G) -> Net-(Q1-C)
- Q1 pad 2: Net-(D1-A) -> Net-(Q1-B)
- Q2 pad 1: BATT+ -> +bat
- Q2 pad 2: BATT+ -> +bat
- Q2 pad 3: BATT+ -> +bat
- Q2 pad 5: +v -> LOAD_IN
- Q2 pad 6: +v -> LOAD_IN
- Q2 pad 7: +v -> LOAD_IN
- Q2 pad 8: +v -> LOAD_IN
- R1 pad 2: Net-(Q1-G) -> Net-(Q1-B)
- R11 pad 1: Net-(J6-Pin_1) -> GND
- R11 pad 2: 6v -> Vsense
- R2 pad 1: Net-(Q1-G) -> LOAD_IN
- R2 pad 2: GND -> Net-(D5-A)
- R4 pad 2: +v -> LOAD
- R5 pad 2: BATT+ -> +bat
- R6 pad 1: Net-(J6-Pin_2) -> Net-(Q1-C)
- R6 pad 2: 6v -> Net-(D5-A)
- U1 pad 20: Net-(U1-AVCC) -> +3v3
- U1 pad 21: unconnected-(U1-AREF-Pad21) -> Net-(U1-AREF)
- U1 pad 23: unconnected-(U1-PC0-Pad23) -> Vsense
- U2 pad 5: IN -> +v
- U5 pad 1: BATT+ -> GND
- U5 pad 2: GND -> +3v3
- U5 pad 3: +3v3 -> +bat
Routing:
- net 1s: track 164.7 -> 58.4 mm
- net Net-(J6-Pin_2): track 62.8 -> 0.00 mm
- net Vsense: track 0.00 -> 60.1 mm
- net Net-(J6-Pin_1): track 44.0 -> 0.00 mm
- net +11.1v: track 104.8 -> 66.5 mm
- net +3v3: track 35.9 -> 12.2 mm, vias 2 -> 0
- net Net-(U4B--): track 23.5 -> 0.00 mm
- net Net-(Q1-G): track 22.7 -> 0.00 mm
- net Net-(U4A-+): track 20.4 -> 0.00 mm
- net Net-(Q1-B): track 0.00 -> 17.9 mm
- net Net-(U4B-+): track 17.5 -> 0.00 mm
- net SCK: track 31.9 -> 17.1 mm
- net Net-(U4A--): track 13.5 -> 0.00 mm
- net Net-(U1-PD7): track 17.9 -> 4.62 mm
- net EN: track 24.0 -> 35.9 mm, vias 0 -> 1
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- added copper zone on F.Cu, net +bat
- added copper zone on In2.Cu, net +v
- added copper zone on F.Cu, net LOAD
- added copper zone on F.Cu, net LOAD_IN
- added copper zone on In1.Cu, net LOAD_IN
- removed copper zone on F.Cu, net +v
- removed copper zone on F.Cu, net 6v
- removed copper zone on F.Cu, net BATT+
- removed copper zone on F.Cu, net IN
- removed copper zone on B.Cu, net Net-(D1-A)
Other:
- copper layers 2 -> 4
- board text removed: "+"
- board text removed: "+3v3"
- board text removed: "<-->"
- board text removed: "EN"
- board text removed: "OutLM393"
- board text removed: "out1 out2"
