File: GPT-E/Schede HW/Files/HeadGPT-E/Head.kicad_pcb (KiCad board)
At the start: 4 copper layers, 81.5 x 81.5 mm, 88 parts, among them J1 Right_Wheel_SERVO, J18 SWITCH, J2 SPEAKER, J3 I2C, J4 Left_Wheel SERVO, J5 Neck_SERVO2, J6 UARTtoRASPI, J7 Neck_SERVO1, J8 FAN, U1 LM3940-3.3, U2 AP64501SP-13, U5 ESP32, U7 MAX98357A, U8 PCA9685PW

Commit message: New file Head v3.0 + production zip
Parts:
- removed C13: 1000uF, Capacitor_THT:CP_Radial_D12.5mm_P5.00mm
- removed C19: 100uF, Capacitor_THT:CP_Radial_D5.0mm_P2.00mm
- removed D9: SS34, Diode_SMD:D_SMA
- removed TP11, TP6: TestPoint, TestPoint:TestPoint_Pad_D1.5mm
- added C14: 100n, Capacitor_SMD:C_0805_2012Metric_Pad1.18x1.45mm_HandSolder, F.Cu at (114.8, 61.6)
- added C20: 10uF, Capacitor_SMD:C_0805_2012Metric_Pad1.18x1.45mm_HandSolder, F.Cu at (115.0, 51.4)
- added C25: 10uF, Capacitor_SMD:C_0805_2012Metric_Pad1.18x1.45mm_HandSolder, F.Cu at (117.2, 51.4)
- added C26: 100n, Capacitor_SMD:C_0805_2012Metric_Pad1.18x1.45mm_HandSolder, F.Cu at (110.9, 61.6)
- added C27: 100p, Capacitor_SMD:C_0805_2012Metric_Pad1.18x1.45mm_HandSolder, F.Cu at (122.7, 66.4)
- added C28: 100n, Capacitor_SMD:C_0805_2012Metric_Pad1.18x1.45mm_HandSolder, F.Cu at (113.5, 55.0)
- added C29: 22u, Capacitor_SMD:C_0805_2012Metric_Pad1.18x1.45mm_HandSolder, F.Cu at (127.9, 57.0)
- added C30: 22u, Capacitor_SMD:C_0805_2012Metric_Pad1.18x1.45mm_HandSolder, F.Cu at (127.9, 59.2)
- added C31: 10uF, Capacitor_SMD:C_0805_2012Metric_Pad1.18x1.45mm_HandSolder, F.Cu at (107.2, 103.6)
- added C32: 10uF, Capacitor_SMD:C_0805_2012Metric_Pad1.18x1.45mm_HandSolder, F.Cu at (109.3, 103.6)
- added L2: 2.2uH, Inductor_SMD:L_Changjiang_FXL0630, F.Cu at (120.9, 58.1)
- added NT1: NetTie_2, NetTie:NetTie-2_SMD_Pad0.5mm, F.Cu at (110.2, 58.5)
- added Q1: AO4407A, Library:SOIC127P600X175-8N, F.Cu at (99.9, 68.0)
- added R27: 249k, Resistor_SMD:R_1206_3216Metric_Pad1.30x1.75mm_HandSolder, F.Cu at (108.8, 54.9)
- added R28: 180k, Resistor_SMD:R_1206_3216Metric_Pad1.30x1.75mm_HandSolder, F.Cu at (122.2, 64.1)
- added R29: 20k, Resistor_SMD:R_1206_3216Metric_Pad1.30x1.75mm_HandSolder, F.Cu at (116.2, 64.1)
- added R30: 10k, Resistor_SMD:R_1206_3216Metric_Pad1.30x1.75mm_HandSolder, F.Cu at (110.7, 64.1)
- added R33: 100k, Resistor_SMD:R_1206_3216Metric_Pad1.30x1.75mm_HandSolder, F.Cu at (107.6, 60.2)
- added U3: TPS56838RPAR, Library:CONV_TPS56838RPAR, F.Cu at (113.4, 58.2)
- C5: value 10uF -> 10nF
- D11: value SMBJ12A -> SMBJ15A
- D5, D6, D7, D8: footprint LED_THT:LED_D5.0mm-4_RGB_Wide_Pins -> Connector:NS-Tech_Grove_1x04_P2mm_Vertical
- R20: value 105k -> 15k8
- moved TP10 59.5 mm to (98.6, 80.2), turned to 90 degrees
- moved J8 57.0 mm to (157.3, 94.6), turned to 180 degrees
- moved R31 53.5 mm to (103.3, 80.1), turned to 180 degrees
- moved C6 50.2 mm to (155.8, 89.8), turned to 0 degrees
- moved R32 50.1 mm to (103.7, 84.7)
- moved C17 42.0 mm to (83.6, 99.0), turned to -90 degrees
- moved J7 37.1 mm to (155.0, 65.6), turned to 180 degrees
- moved C9 33.3 mm to (121.0, 110.5), turned to 90 degrees
- moved J5 31.4 mm to (147.4, 51.9), turned to 0 degrees
- moved TP1 26.2 mm to (83.6, 95.3)
- moved J6 17.0 mm to (155.8, 110.4), turned to 90 degrees
- moved C18 15.5 mm to (93.0, 68.1)
- moved F1 11.8 mm to (101.3, 58.4), turned to -90 degrees
- moved J2 11.6 mm to (84.7, 119.8), turned to 90 degrees
- moved TP5 11.6 mm to (85.2, 105.5)
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Connections:
- net 11.1v renamed Battery
- C15 pad 1: +5V -> +6v
- C18 pad 1: Net-(D11-K) -> Net-(J18-Pin_1)
- C9 pad 1: +3v3 -> +5V
- F1 pad 1: Net-(D9-K) -> Net-(D11-K)
- F1 pad 2: Net-(J18-Pin_1) -> Net-(F1-Pad2)
- J1 pad 2: +5V -> +6v
- J1 pad 3: PWM12 -> RWheel_Servo
- J4 pad 2: +5V -> +6v
- J4 pad 3: PWM13 -> LWheel_Servo
- J5 pad 2: +5V -> +6v
- J5 pad 3: PWM15 -> Neck_S2
- J7 pad 2: +5V -> +6v
- J7 pad 3: PWM14 -> Neck_S1
- U5 pad 1: unconnected-(U5-VIN-Pad1) -> +5V
- U5 pad 12: unconnected-(U5-D34-Pad12) -> SERVO_PWR_GOOD
- U5 pad 16: unconnected-(U5-D23-Pad16) -> Neck_S1
- U5 pad 21: unconnected-(U5-D19-Pad21) -> Neck_S2
- U5 pad 22: unconnected-(U5-D18-Pad22) -> LWheel_Servo
- U5 pad 23: UART_TX -> unconnected-(U5-D5-Pad23)
- U5 pad 24: unconnected-(U5-TX2-Pad24) -> RWheel_Servo
- U5 pad 26: unconnected-(U5-D4-Pad26) -> SERVO_PWR_EN
- U5 pad 3: unconnected-(U5-D13-Pad3) -> UART_TX
- U5 pad 30: +3v3 -> unconnected-(U5-3V3-Pad30)
- U8 pad 19: PWM12 -> unconnected-(U8-LED12-Pad19)
- U8 pad 20: PWM13 -> unconnected-(U8-LED13-Pad20)
- U8 pad 21: PWM14 -> unconnected-(U8-LED14-Pad21)
- U8 pad 22: PWM15 -> unconnected-(U8-LED15-Pad22)
Routing:
- net +5V: track 112.1 -> 24.0 mm
- net SERVO_PWR_EN: track 0.00 -> 75.7 mm, vias 0 -> 1
- net PWM14: track 50.1 -> 0.00 mm
- net LWheel_Servo: track 0.00 -> 46.9 mm
- net Neck_S2: track 0.00 -> 44.5 mm
- net PWM13: track 43.6 -> 0.00 mm
- net PWM15: track 41.2 -> 0.00 mm
- net RWheel_Servo: track 0.00 -> 38.4 mm
- net SERVO_PWR_GOOD: track 0.00 -> 34.0 mm, vias 0 -> 1
- net PWM12: track 31.8 -> 0.00 mm
- net UART_TX: track 5.85 -> 34.6 mm
- net Net-(U3-AGND): track 0.00 -> 22.8 mm, vias 0 -> 2
- net Net-(U3-FB): track 0.00 -> 16.2 mm
- net Net-(D11-K): track 0.00 -> 14.0 mm
- net +3v3: track 8.40 -> 20.8 mm, vias 11 -> 14
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- added copper zone on F.Cu, net +6v
- added copper zone on In2.Cu, net +6v
- added copper zone on F.Cu, net Battery
- added copper zone on In2.Cu, net Battery
- removed copper zone on F.Cu, net Net-(D11-K)
