File: GPT-E/Schede HW/Files/HeadGPT-E/Head.kicad_sch (KiCad schematic)
At the start: 88 parts, among them J1 Right_Wheel_SERVO, J18 SWITCH, J2 SPEAKER, J3 I2C, J4 Left_Wheel SERVO, J5 Neck_SERVO2, J6 UARTtoRASPI, J7 Neck_SERVO1, J8 FAN, U1 LM3940-3.3, U2 AP64501SP-13, U5 ESP32, U7 MAX98357A, U8 PCA9685PW

Commit message: New file Head v3.0 + production zip
Parts:
- removed C13: 1000uF, Capacitor_THT:CP_Radial_D12.5mm_P5.00mm, symbol Device:C_Polarized
- removed C19: 100uF, Capacitor_THT:CP_Radial_D5.0mm_P2.00mm, symbol Device:C_Polarized
- removed D9: SS34, Diode_SMD:D_SMA, symbol Diode:SS34
- removed TP11, TP6: TestPoint, TestPoint:TestPoint_Pad_D1.5mm, symbol Connector:TestPoint
- added C14, C28: 100n, Capacitor_SMD:C_0805_2012Metric_Pad1.18x1.45mm_HandSolder, symbol Device:C
- added C20, C25, C31, C32: 10uF, Capacitor_SMD:C_0805_2012Metric_Pad1.18x1.45mm_HandSolder, symbol Device:C
- added C26: DNP, Capacitor_SMD:C_0805_2012Metric_Pad1.18x1.45mm_HandSolder, symbol Device:C
- added C27: 100p, Capacitor_SMD:C_0805_2012Metric_Pad1.18x1.45mm_HandSolder, symbol Device:C
- added C29, C30: 22u, Capacitor_SMD:C_0805_2012Metric_Pad1.18x1.45mm_HandSolder, symbol Device:C
- added L2: 2.2uH, Inductor_SMD:L_Changjiang_FXL0630, symbol Device:L
- added NT1: NetTie_2, NetTie:NetTie-2_SMD_Pad0.5mm, symbol Device:NetTie_2
- added Q1: AO4407A, Library:SOIC127P600X175-8N, symbol Libreria_Personale:AO4407A
- added R27: DNP, Resistor_SMD:R_1206_3216Metric_Pad1.30x1.75mm_HandSolder, symbol Device:R
- added R28: 180k, Resistor_SMD:R_1206_3216Metric_Pad1.30x1.75mm_HandSolder, symbol Device:R
- added R29: 20k, Resistor_SMD:R_1206_3216Metric_Pad1.30x1.75mm_HandSolder, symbol Device:R
- added R30: 10k, Resistor_SMD:R_1206_3216Metric_Pad1.30x1.75mm_HandSolder, symbol Device:R
- added R33: 100k, Resistor_SMD:R_1206_3216Metric_Pad1.30x1.75mm_HandSolder, symbol Device:R
- added U3: TPS56838RPAR, Library:CONV_TPS56838RPAR, symbol Libreria_Personale:TPS56838RPAR
- C5: value 10uF -> 10nF
- D11: value SMBJ12A -> SMBJ15A
- D5, D6, D7, D8: footprint LED_THT:LED_D5.0mm-4_RGB_Wide_Pins -> Connector:NS-Tech_Grove_1x04_P2mm_Vertical
- R20: value 105k -> 15k8
Connections:
- net +3v3: now also C31.1, C32.1, R30.2; no longer C9.1, U5.30 (3V3)
- net +5V: now also C9.1, U5.1 (VIN); no longer C15.1, J1.2 (Pin_2), J4.2 (Pin_2), J5.2 (Pin_2), J7.2 (Pin_2)
- net GND: now also C20.2, C25.2, C28.1, C29.2, C30.2, C31.2, C32.2, NT1.1, Q1.4, U3.9 (PGND)
- net UART_TX: now also U5.3 (D13); no longer U5.23 (D5)
- net at J18.1 (Pin_1): now also C18.1, Q1.1, Q1.2, Q1.3; no longer F1.2
- net at D11.1 (K), J23.2 (+), J23.4 (+): now also F1.1; no longer C18.1
- net SERVO_PWR_GOOD: now reaches U5.12 (D34)
- net SERVO_PWR_GOOD: now also R30.1, U3.4 (PG)
- net Neck_S1: now reaches U5.16 (D23)
- net Neck_S1: now also J7.3 (Pin_3)
- net Neck_S2: now reaches U5.21 (D19)
- net Neck_S2: now also J5.3 (Pin_3)
- net LWheel_Servo: now reaches U5.22 (D18)
- net LWheel_Servo: now also J4.3 (Pin_3)
- net RWheel_Servo: now reaches U5.24 (TX2)
- net RWheel_Servo: now also J1.3 (Pin_3)
- net SERVO_PWR_EN: now reaches U5.26 (D4)
- net SERVO_PWR_EN: now also R33.1, U3.1 (EN)
- net 11.1v renamed Battery
- net Battery: now also C20.1, C25.1, C28.2, U3.8 (VIN)
- net PWM12: no longer names the net of U8.19 (LED12)
- net PWM12: no longer J1.3 (Pin_3)
- net PWM13: no longer names the net of U8.20 (LED13)
- net PWM13: no longer J4.3 (Pin_3)
- net PWM14: no longer names the net of U8.21 (LED14)
- net PWM14: no longer J7.3 (Pin_3)
- net PWM15: no longer names the net of U8.22 (LED15)
- net PWM15: no longer J5.3 (Pin_3)
- new net: C26.2, NT1.2, R27.1, R29.2, R33.2, U3.3 (AGND)
- new net: R27.2, U3.10 (MODE)
- new net: C27.2, R28.2, R29.1, U3.2 (FB)
- new net: C26.1, U3.5 (SS)
- new net: C14.2, L2.1, U3.6 (SW)
- new net: C14.1, U3.7 (BOOT)
- new net: F1.2, Q1.5, Q1.6, Q1.7, Q1.8
- new net +6v: C15.1, C27.1, C29.1, C30.1, J1.2 (Pin_2), J4.2 (Pin_2), J5.2 (Pin_2), J7.2 (Pin_2), L2.2, R28.1
- no-connect marks 15 -> 13
Other:
- moved on the sheet: C15, C18, C2, C3, C8, C9, D11, F1, J1, J18, J23, J4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
